File: pic/pic.brd (EAGLE design)
At the start: 80 x 100 mm, 51 parts, among them IC1 PIC16F877P, IC4 7805T, IC5 MAX233, IC7 PCA82C250, Q2 200MHz, Q3 16MHz, U1 MCP2510P

Commit message: Updated board
Parts:
- moved R11 159.5 mm to (45.0, 24.5)
- moved R24 127.6 mm to (70.4, 58.7)
- moved R16 126.1 mm to (58.3, 58.5)
- moved R22 122.8 mm to (83.3, 71.4), turned to 180 degrees
- moved R15 122.2 mm to (70.6, 67.9)
- moved LED8 119.1 mm to (15.4, 76.1), turned to 270 degrees
- moved LED13 118.2 mm to (95.1, 57.8)
- moved LED7 112.2 mm to (95.6, 17.8)
- moved R21 109.8 mm to (83.2, 74.2), turned to 180 degrees
- moved J1 104.7 mm to (89.2, 11.2), turned to 90 degrees
- moved C1 102.4 mm to (72.9, 72.8), turned to 180 degrees
- moved C2 101.8 mm to (64.8, 72.9), turned to 180 degrees
- moved R17 101.0 mm to (18.5, 60.3), turned to 270 degrees
- moved C7 95.2 mm to (38.0, 69.7)
- moved C5 90.9 mm to (43.7, 69.6)
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Routing:
- net GND: track 0.00 -> 424.0 mm, vias 0 -> 1
- net VCC: track 0.00 -> 393.3 mm, vias 0 -> 2
- net C6: track 0.00 -> 217.5 mm, vias 0 -> 2
- net B7: track 0.00 -> 194.6 mm, vias 0 -> 2
- net RESET: track 0.00 -> 183.9 mm
- net OSC2: track 0.00 -> 172.2 mm, vias 0 -> 6
- net D1: track 0.00 -> 170.2 mm
- net B4: track 0.00 -> 149.5 mm, vias 0 -> 8
- net N$10: track 0.00 -> 145.1 mm, vias 0 -> 3
- net A4: track 0.00 -> 144.4 mm, vias 0 -> 2
- net C7: track 0.00 -> 140.1 mm, vias 0 -> 6
- net OSC1: track 0.00 -> 137.1 mm, vias 0 -> 7
- net B6: track 0.00 -> 112.1 mm, vias 0 -> 4
- net B0: track 0.00 -> 111.6 mm, vias 0 -> 2
- net N$38: track 0.00 -> 100.7 mm, vias 0 -> 2
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Other:
- board size 80 x 100 mm -> 100 x 80 mm
